Commit message: Reorganize camera code; add slider interface; WIP wrist camera not following robot wrist

File: pybullet-playground_2/urdf/pybullet_ur5_gripper/robots/urdf/ur5e.urdf (robot description, URDF)
Before this commit: robot ur5e, 12 links, 11 joints
Links:
- added link wrist_camera_link; visual sphere radius=0.03
Joints:
- added joint wrist_camera_joint: type fixed, parent baseLink, child wrist_camera_link, origin xyz=0 -0.05 0 rpy=0 0 0

Commit message: Add wrist cam rgb virtual cam rendering

File: pybullet-playground_2/urdf/pybullet_ur5_gripper/robots/urdf/ur5e.urdf (robot description, URDF)
Before this commit: robot ur5e, 13 links, 12 joints
Links:
- added link wrist_camera_vis_x_link; visual cylinder length=0.1 radius=0.005
- added link wrist_camera_vis_y_link; visual cylinder length=0.1 radius=0.005
- added link wrist_camera_vis_z_link; visual cylinder length=0.1 radius=0.005
- link wrist_camera_link: geometry 
Joints:
- removed joint wrist_camera_joint
- added joint wrist_camera_vis_joint: type fixed, parent baseLink, child wrist_camera_link, origin xyz=0 -0.1 0.05 rpy=0 0 0
- added joint wrist_camera_vis_x_joint: type fixed, parent wrist_camera_link, child wrist_camera_vis_x_link, origin xyz=0 0 0 rpy=0 0 0
- added joint wrist_camera_vis_y_joint: type fixed, parent wrist_camera_link, child wrist_camera_vis_y_link, origin xyz=0 0 0 rpy=0 0 0
- added joint wrist_camera_vis_z_joint: type fixed, parent wrist_camera_link, child wrist_camera_vis_z_link, origin xyz=0 0 0 rpy=0 0 0
